File: 833iot.kicad_sch (KiCad schematic)
At the start: 24 parts, among them J1 U254-051T-4BH83-F1S, J2 Conn_01x04, J3 Conn_01x02, J4 Conn_01x15_Male, J5 Conn_01x15_Male, Q1 AO3407, Q2 AO3407, SW1 SW_SPST, U1 E73-2G4M08S1E, U2 AP2112K-3.3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

Commit message: fix vias issue
Parts:
- D2: value BLUE -> Yellow; LCSC Part # C273617 -> C74343
- D3: LCSC Part # C264458 -> C253533
- D4: value PURPLE -> Green; LCSC Part # C264473 -> C181862
- J1: LCSC Part # (none) -> C397452
Changed lines of the file:
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@@
     (in_bom yes) (on_board yes)
     (property "Reference" "D2" (id 0) (at 52.2478 106.553 0))
-    (property "Value" "BLUE" (id 1) (at 52.2478 108.8644 0))
+    (property "Value" "Yellow" (id 1) (at 52.2478 108.8644 0))
     (property "Footprint" "LED_SMD:LED_0603_1608Metric" (id 2) (at 52.07 113.03 0)
       (effects (font (size 1.27 1.27)) hide)
@@
       (effects (font (size 1.27 1.27)) hide)
     )
-    (property "LCSC Part #" "C273617" (id 4) (at 52.07 113.03 0)
+    (property "LCSC Part #" "C74343" (id 4) (at 52.07 113.03 0)
       (effects (font (size 1.27 1.27)) hide)
     )
@@
     (property "PARTREV" "A0" (id 7) (at 254 36.83 0)
       (effects (font (size 1.27 1.27)) (justify left bottom) hide)
+    )
+    (property "LCSC Part #" "C397452" (id 8) (at 254 36.83 0)
+      (effects (font (size 1.27 1.27)) hide)
     )
     (pin "1")
@@
       (effects (font (size 1.27 1.27)) hide)
     )
-    (property "LCSC Part #" "C264458" (id 4) (at 109.22 164.465 0)
+    (property "LCSC Part #" "C253533" (id 4) (at 109.22 164.465 0)
       (effects (font (size 1.27 1.27)) hide)
     )
@@
     (in_bom yes) (on_board yes)
     (property "Reference" "D4" (id 0) (at 52.2478 119.253 0))
-    (property "Value" "PURPLE" (id 1) (at 52.2478 121.5644 0))
+    (property "Value" "Green" (id 1) (at 52.2478 121.5644 0))
     (property "Footprint" "LED_SMD:LED_0603_1608Metric" (id 2) (at 52.07 125.73 0)
       (effects (font (size 1.27 1.27)) hide)
@@
       (effects (font (size 1.27 1.27)) hide)
     )
-    (property "LCSC Part #" "C264473" (id 4) (at 52.07 125.73 0)
+    (property "LCSC Part #" "C181862" (id 4) (at 52.07 125.73 0)
       (effects (font (size 1.27 1.27)) hide)
     )
@@
     )
     (path "/00000000-0000-0000-0000-00005eb6247d"
-      (reference "D2") (unit 1) (value "BLUE") (footprint "LED_SMD:LED_0603_1608Metric")
+      (reference "D2") (unit 1) (value "Yellow") (footprint "LED_SMD:LED_0603_1608Metric")
     )
     (path "/6417a26b-7fa3-4f15-9e1b-9d747117c266"
@@
     )
     (path "/c3a908c6-01d5-471a-9374-ecf08b2430e4"
-      (reference "D4") (unit 1) (value "PURPLE") (footprint "LED_SMD:LED_0603_1608Metric")
+      (reference "D4") (unit 1) (value "Green") (footprint "LED_SMD:LED_0603_1608Metric")
     )
     (path "/074cc084-3be5-43a7-9756-c42bb82c7ad7"
